Commit message: ragaceebi viwvale

File: description/robot.urdf.xacro (robot description, xacro)
@@ -2,3 +2,4 @@
 <robot xmlns:xacro="http://www.ros.org/wiki/xacro"  name="robot">
    <xacro:include filename="robot_core.xacro" />
+   <xacro:include filename="gazebo_control.xacro" />
 </robot>

File: description/robot_core.xacro (robot description, xacro)
@@ -34,8 +34,11 @@
             </geometry>
         </collision>
-        <xacro:inertial_box mass="70" x="1.13" y="0.46" z="0.45">]
+        <xacro:inertial_box mass="1" x="1.13" y="0.46" z="0.45">]
             <origin xyz="0.56 0 0.225" rpy="0 0 0"/>
         </xacro:inertial_box>
     </link>
+    <gazebo reference="chassis">
+        <material> Gazebo/Blue </material>
+    </gazebo>
     <!-- LEFT WHEEL LINK -->
      <joint name="left_wheel_joint" type="continuous">
@@ -48,5 +51,5 @@
          <visual>
             <geometry>
-                <cylinder radius="0.10" length="0.07"/>
+                <cylinder radius="0.30" length="0.07"/>
             </geometry>
            <material name="black"/>
@@ -54,11 +57,14 @@
           <collision>
             <geometry>
-                <cylinder radius="0.10" length="0.07"/>
+                <cylinder radius="0.30" length="0.07"/>
             </geometry>
          </collision>
-          <xacro:inertial_cylinder mass="10" length="0.07" radius="0.10">]
+          <xacro:inertial_cylinder mass="1" length="0.07" radius="0.30">]
             <origin xyz="0 0 0" rpy="0 0 0"/>
           </xacro:inertial_cylinder>
     </link>
+    <gazebo reference="left_wheel">
+        <material> Gazebo/Black </material>
+    </gazebo>
  <!-- RIGHT WHEEL LINK -->
      <joint name="right_wheel_joint" type="continuous">
@@ -71,5 +77,5 @@
          <visual>
             <geometry>
-                <cylinder radius="0.10" length="0.07"/>
+                <cylinder radius="0.30" length="0.07"/>
             </geometry>
            <material name="black"/>
@@ -77,11 +83,14 @@
          <collision>
             <geometry>
-                <cylinder radius="0.10" length="0.07"/>
+                <cylinder radius="0.30" length="0.07"/>
             </geometry>
          </collision>
-         <xacro:inertial_cylinder mass="10" length="0.07" radius="0.10">]
+         <xacro:inertial_cylinder mass="1" length="0.07" radius="0.30">]
             <origin xyz="0 0 0" rpy="0 0 0"/>
           </xacro:inertial_cylinder>
     </link>
+    <gazebo reference="right_wheel">
+        <material> Gazebo/Black </material>
+    </gazebo>
 <!--CASTER WHEEL LINK-->
  <joint name="caste_wheel_joint" type="fixed">
@@ -106,3 +115,6 @@
           </xacro:inertial_sphere>
     </link>
+    <gazebo reference="caster_wheel">
+        <material> Gazebo/Black </material>
+    </gazebo>
 </robot>
